Commit message: Working cloud map for the realsense cam on the UR3e

File: universal_robot/ur_gazebo/urdf/urRealSense.xacro (robot description, xacro)
@@ -73,7 +73,7 @@
     a 'world' link there.
   -->
-  <link name="world"/>
-  <joint name="world_joint" type="fixed">
-    <parent link="world"/>
+  <link name="/map"/>
+  <joint name="mpa_joint" type="fixed">
+    <parent link="/map"/>
     <child link="base_link"/>
     <origin xyz="0 0 0" rpy="0 0 0"/>

Commit message: New point cloud render for Realsense with Rtabmap, waiting to be tested with a working tf (aka tested on the real UR3e)

File: universal_robot/ur_gazebo/urdf/urRealSense.xacro (robot description, xacro)
@@ -1,4 +1,4 @@
 <?xml version="1.0"?>
-<robot xmlns:xacro="http://wiki.ros.org/xacro" name="$(arg robot_model)_robot">
+<robot xmlns:xacro="http://wiki.ros.org/xacro" name="ur3e_robot">
   <!--
     This is a top-level xacro instantiating the Gazebo-specific version of the
@@ -73,7 +73,7 @@
     a 'world' link there.
   -->
-  <link name="/map"/>
-  <joint name="mpa_joint" type="fixed">
-    <parent link="/map"/>
+  <link name="world"/>
+  <joint name="world_joint" type="fixed">
+    <parent link="world"/>
     <child link="base_link"/>
     <origin xyz="0 0 0" rpy="0 0 0"/>
@@ -149,5 +149,5 @@
     <parent link="tool0_controller"/>
     <child link="multispec_cam"/>
-    <origin xyz="+0.045 +0.030 0" rpy="0 0 0"/>
+    <origin xyz="+0.045 +0.030 0.0" rpy="0 0 0"/>
   </joint>
   </xacro:macro>

Commit message: Camera support offset adjusted and demo3.launch set to take simulation  as an argument (sim) to be used as well for real montage

File: universal_robot/ur_gazebo/urdf/urRealSense.xacro (robot description, xacro)
@@ -113,5 +113,5 @@
     <parent link="tool0_controller"/>
     <child link="camera_support_link"/>
-    <origin xyz="0 -0.04 0" rpy="${pi/2} ${pi} ${pi}"/>
+    <origin xyz="0 -0.055 0" rpy="${pi/2} ${pi} ${pi}"/>
   </joint>
   <xacro:sensor_d435i

Commit message: Transfert to industrial computer

File: universal_robot/ur_gazebo/urdf/urRealSense.xacro (robot description, xacro)
@@ -113,5 +113,5 @@
     <parent link="tool0_controller"/>
     <child link="camera_support_link"/>
-    <origin xyz="0 -0.055 0" rpy="${pi/2} ${pi} ${pi}"/>
+    <origin xyz="0 -0.055 ${-0.026+0.02}" rpy="${pi/2} ${pi} ${pi}"/>
   </joint>
   <xacro:sensor_d435i
