Commit message: Try to merge the models of ur3e and realsense camera, the base_link of the lowest xacro has been renamed though. Think to change it or find a solution to not generate a base_link in the realsense2_description

File: universal_robot/ur_description/urdf/inc/ur_macro.xacro (robot description, xacro)
@@ -64,5 +64,5 @@
     <xacro:ur_arm_transmission prefix="${prefix}" hw_interface="${transmission_hw_interface}" />
     <!-- links: main serial chain -->
-    <link name="${prefix}base_link"/>
+    <link name="${prefix}dbase_link"/>
     <link name="${prefix}base_link_inertia">
       <visual>
@@ -208,5 +208,5 @@
     <!-- joints: main serial chain -->
     <joint name="${prefix}base_link-base_link_inertia" type="fixed">
-      <parent link="${prefix}base_link" />
+      <parent link="${prefix}dbase_link" />
       <child link="${prefix}base_link_inertia" />
       <!-- 'base_link' is REP-103 aligned (so X+ forward), while the internal
@@ -298,5 +298,5 @@
       -->
       <origin xyz="0 0 0" rpy="0 0 ${pi}"/>
-      <parent link="${prefix}base_link"/>
+      <parent link="${prefix}dbase_link"/>
       <child link="${prefix}base"/>
     </joint>

Commit message: Mapping with realsense on the ur3e arm, but the point map cannot be visualized in Rviz if the arm is simulated due to tf publication rate issues

File: universal_robot/ur_description/urdf/inc/ur_macro.xacro (robot description, xacro)
@@ -64,5 +64,5 @@
     <xacro:ur_arm_transmission prefix="${prefix}" hw_interface="${transmission_hw_interface}" />
     <!-- links: main serial chain -->
-    <link name="${prefix}dbase_link"/>
+    <link name="${prefix}base_link"/>
     <link name="${prefix}base_link_inertia">
       <visual>
@@ -208,5 +208,5 @@
     <!-- joints: main serial chain -->
     <joint name="${prefix}base_link-base_link_inertia" type="fixed">
-      <parent link="${prefix}dbase_link" />
+      <parent link="${prefix}base_link" />
       <child link="${prefix}base_link_inertia" />
       <!-- 'base_link' is REP-103 aligned (so X+ forward), while the internal
@@ -298,5 +298,5 @@
       -->
       <origin xyz="0 0 0" rpy="0 0 ${pi}"/>
-      <parent link="${prefix}dbase_link"/>
+      <parent link="${prefix}base_link"/>
       <child link="${prefix}base"/>
     </joint>

File: universal_robot/ur_gazebo/urdf/urRealSense.xacro (robot description, xacro)
@@ -25,5 +25,5 @@
   -->
   <xacro:include filename="$(find ur_gazebo)/urdf/ur_macro.xacro"/>
-  <xacro:include filename='$(find realsense2_description)/urdf/test_d435i_camera.urdf.xacro'/>
+  <xacro:include filename="$(find realsense2_description)/urdf/_d435i.urdf.xacro"/>
   <!--Declare arguments -->
   <xacro:arg name="joint_limit_params" default=""/>
@@ -43,4 +43,15 @@
   <xacro:arg name="safety_pos_margin" default="0.15"/>
   <xacro:arg name="safety_k_position" default="20"/>
+  <xacro:macro name="ur_realsense" params="
+    prefix
+    joint_limits_parameters_file:=$(arg joint_limit_params)
+    kinematics_parameters_file:=$(arg kinematics_params)
+    physical_parameters_file:=$(arg physical_params)
+    visual_parameters_file:=$(arg visual_params)
+    transmission_hw_interface:=$(arg transmission_hw_interface)
+    safety_limits:=$(arg safety_limits)
+    safety_pos_margin:=$(arg safety_pos_margin)
+    safety_k_position:=$(arg safety_k_position)"
+  >
   <!-- Instantiate the Gazebo robot and pass it all the required arguments. -->
   <xacro:ur_robot_gazebo
@@ -68,9 +79,9 @@
     <origin xyz="0 0 0" rpy="0 0 0"/>
   </joint>
-  <joint name="base_wjoint" type="fixed">
+  <!--joint name="base_wjoint" type="fixed">
     <parent link="base_link"/>
     <child link="dbase_link"/>
     <origin xyz="0 0 0" rpy="0 0 0"/>
-  </joint>
+  </joint-->
   <link name="tool0_controller"/>
   <joint name="tool_controller_fake_joint" type="fixed">
@@ -105,5 +116,5 @@
   </joint>
   <xacro:sensor_d435i
-    name="cam1"
+    name="camera"
     parent="camera_support_link"
     use_nominal_extrinsics="true">
@@ -140,3 +151,4 @@
     <origin xyz="+0.045 +0.030 0" rpy="0 0 0"/>
   </joint>
+  </xacro:macro>
 </robot>
