Commit message: Simulator reworking thanks to merging universal_robots with previous versions

File: universal_robot/ur_description/urdf/inc/gripper.xacro (robot description, xacro)
@@ -17,5 +17,5 @@
     physical_parameters_file
     visual_parameters_file
-    transmission_hw_interface:=hardware_interface/EffortJointInterface
+    transmission_hw_interface:=hardware_interface/PositionJointInterface
     safety_limits:=false
     safety_pos_margin:=0.15
@@ -50,5 +50,5 @@
         </geometry>
       </collision>
-      <xacro:cylinder_inertial radius="0.01" length="0.01" mass="0.01"><!--${wrist_3_inertia_radius}" length="${wrist_3_inertia_length}"  mass="${wrist_3_mass}"-->
+      <xacro:cylinder_inertial radius="0.05" length="0.1" mass="0.1">
         <origin xyz="0 0 0" rpy="0 0 0" />
       </xacro:cylinder_inertial>

File: universal_robot/ur_description/urdf/inc/ur5_macro.xacro (robot description, xacro)
@@ -28,5 +28,5 @@
    safety_k_position:=20"
   >
-    <xacro:include filename="$(find ur_description)/urdf/inc/ur_macro.xacro"/>
+    <xacro:include filename="$(find ur_description)/urdf/inc/ur_macro_mod.xacro"/>
     <xacro:ur_robot
       prefix="${prefix}"

File: universal_robot/ur_description/urdf/inc/ur5_macro_g.xacro (robot description, xacro)
@@ -28,5 +28,5 @@
    safety_k_position:=20"
   >
-    <xacro:include filename="$(find ur_description)/urdf/inc/gripper.xacro"/>
+    <!--xacro:include filename="$(find ur_description)/urdf/inc/gripper.xacro"/>
     <xacro:gripper
       prefix="${prefix}"
@@ -39,5 +39,17 @@
       safety_pos_margin="${safety_pos_margin}"
       safety_k_position="${safety_k_position}"
-    />
+    /-->
+    <xacro:include filename="$(find summit_xl_hl_ur5_description)/robots/summit_xl_hl_ur5.urdf.xacro"/>
+    <xacro:summit_robot
+   prefix="${prefix}"
+   joint_limits_parameters_file='${joint_limits_parameters_file}'
+   kinematics_parameters_file='${kinematics_parameters_file}'
+   physical_parameters_file='${physical_parameters_file}'
+   visual_parameters_file='${visual_parameters_file}'
+   transmission_hw_interface='${transmission_hw_interface}'
+   safety_limits="${safety_limits}"
+   safety_pos_margin="${safety_pos_margin}"
+   safety_k_position="${safety_k_position}"
+  />
   </xacro:macro>
 </robot>

File: universal_robot/ur_description/urdf/ur5_g.xacro (robot description, xacro)
@@ -15,4 +15,4 @@
   -->
   <xacro:include filename="$(find ur_description)/urdf/inc/ur5_macro_g.xacro"/>
-  <xacro:ur5_robot prefix="" />
+  <xacro:ur5_robot prefix="arm_" />
 </robot>

File: universal_robot/ur_gazebo/urdf/ur.xacro (robot description, xacro)
@@ -30,4 +30,5 @@
   <xacro:arg name="kinematics_params" default=""/>
   <xacro:arg name="visual_params" default=""/>
+  <xacro:arg name="prefix" default=""/>
   <!--
     legal values:
@@ -44,5 +45,5 @@
   <!-- Instantiate the Gazebo robot and pass it all the required arguments. -->
   <xacro:ur_robot_gazebo
-    prefix=""
+    prefix="$(arg prefix)"
     joint_limits_parameters_file="$(arg joint_limit_params)"
     kinematics_parameters_file="$(arg kinematics_params)"
@@ -61,15 +62,69 @@
     a 'world' link there.
   -->
-  <link name="world"/>
+  <!--link name="world"/>
   <joint name="world_joint" type="fixed">
     <parent link="world"/>
-    <child link="base_link"/>
+    <child link="$(arg prefix)base_link"/>
     <origin xyz="0 0 0" rpy="0 0 0"/>
-  </joint>
+  </joint-->
   <link name="tool0_controller"/>
   <joint name="tool_controller_fake_joint" type="fixed">
-    <parent link="tool0"/>
+    <parent link="$(arg prefix)tool0"/>
     <child link="tool0_controller"/>
     <origin xyz="0 0 0" rpy="0 0 0"/>
   </joint>
+  <joint name="camera_optical_joint" type="fixed">
+    <parent link="camera_link"/>
+    <child link="camera_link_optical"/>
+    <origin xyz="0 0 0.1" rpy="0 ${-pi/2} ${-pi/2}"/>
+  </joint>
+  <link name="camera_link_optical"/>
+  <gazebo reference="camera_link_optical">
+    <sensor type="camera" name="camera1">
+    <pose> 0 0 0 0 0 0 </pose>
+      <update_rate>30.0</update_rate>
+      <visualize>true</visualize>
+      <camera name="head">
+        <horizontal_fov>1.3962634</horizontal_fov>
+        <image>
+          <width>800</width>
+          <height>800</height>
+          <format>R8G8B8</format>
+        </image>
+        <clip>
+          <near>0.02</near>
+          <far>300</far>
+        </clip>
+        <noise>
+          <type>gaussian</type>
+          <!-- Noise is sampled independently per pixel on each frame.
+               That pixel's noise value is added to each of its color
+               channels, which at that point lie in the range [0,1]. -->
+          <mean>0.0</mean>
+          <stddev>0.007</stddev>
+        </noise>
+      </camera>
+      <plugin name="camera_controller" filename="libgazebo_ros_camera.so">
+        <alwaysOn>true</alwaysOn>
+        <updateRate>0.0</updateRate>
+        <cameraName>camera1</cameraName>
+        <imageTopicName>image_raw</imageTopicName>
+        <cameraInfoTopicName>camera_info</cameraInfoTopicName>
+        <frameName>camera_link_optical</frameName>
+        <!-- setting hackBaseline to anything but 0.0 will cause a misalignment
+            between the gazebo sensor image and the frame it is supposed to
+            be attached to -->
+        <hackBaseline>0.0</hackBaseline>
+        <distortionK1>0.0</distortionK1>
+        <distortionK2>0.0</distortionK2>
+        <distortionK3>0.0</distortionK3>
+        <distortionT1>0.0</distortionT1>
+        <distortionT2>0.0</distortionT2>
+        <CxPrime>0</CxPrime>
+        <Cx>0.0</Cx>
+        <Cy>0.0</Cy>
+        <focalLength>0.0</focalLength>
+      </plugin>
+    </sensor>
+  </gazebo>
 </robot>

File: universal_robot/ur_gazebo/urdf/ur_macro.xacro (robot description, xacro)
@@ -46,7 +46,7 @@
       the definitions for the real robot.
     -->
-  <xacro:include filename="$(find ur_description)/urdf/inc/ur_macro.xacro"/>
+  <xacro:include filename="$(find summit_xl_hl_ur5_description)/robots/summit_xl_hl_ur5.urdf.xacro"/>
     <!-- Instantiate model for the REAL robot. -->
-    <xacro:ur_robot
+    <!--xacro:ur_robot
       prefix="${prefix}"
       joint_limits_parameters_file="${joint_limits_parameters_file}"
@@ -58,5 +58,16 @@
       safety_pos_margin="${safety_pos_margin}"
       safety_k_position="${safety_k_position}"
-    />
+    /-->
+    <xacro:summit_robot
+   prefix="${prefix}"
+   joint_limits_parameters_file='${joint_limits_parameters_file}'
+   kinematics_parameters_file='${kinematics_parameters_file}'
+   physical_parameters_file='${physical_parameters_file}'
+   visual_parameters_file='${visual_parameters_file}'
+   transmission_hw_interface='${transmission_hw_interface}'
+   safety_limits="${safety_limits}"
+   safety_pos_margin="${safety_pos_margin}"
+   safety_k_position="${safety_k_position}"
+  />
     <!-- Configure self collision properties per link -->
     <gazebo reference="${prefix}shoulder_link">
